Commit message: fix: get headless Gazebo sim SLAM pipeline fully working
- docker/Dockerfile: add ENABLE_HW_STACK=0 arg, make hw deps conditional
- docker/entrypoint.sh: add LIBGL_ALWAYS_SOFTWARE=1 + MESA_GL_VERSION_OVERRIDE
  for headless ogre rendering (enables gpu_lidar sensor without a GPU)
- docker-compose.yml: align RMW to rmw_cyclonedds_cpp for sim+rviz services
- docker-compose.hw.yml: set ENABLE_HW_STACK=1 for hardware image builds
- src/g1_description/g1_23dof.urdf:
  - add base_footprint link + fixed joint (required by Nav2/SLAM)
  - add lidar_link + fixed joint at pelvis+0.3m
  - add gpu_lidar sensor (360deg, 16 beams, 10Hz, topic /lidar/points)
  - add OdometryPublisher plugin (odom->base_footprint TF + /odom)
  - add VelocityControl plugin (/cmd_vel)
  - fix all 50 mesh paths: meshes/ -> package://g1_description/meshes/
- src/g1_gazebo/worlds/indoor_office.sdf:
  - fix plugin names: gz:: -> ignition::gazebo::systems:: with correct .so filenames
  - change render_engine from ogre2 to ogre (CPU, works headless with Mesa)
- src/g1_gazebo/launch/sim_all.launch.py:
  - fix bridge: /lidar/points/points (PointCloudPacked) not /lidar/points (LaserScan)
  - add /tf bridge (ignition.msgs.Pose_V)
  - add inline pointcloud_to_laserscan node
  - set RELIABLE QoS on /scan publisher so slam_toolbox+Nav2 can subscribe
  - spawn robot via -topic /robot_description instead of -string
  - remove redundant static TF odom->base_footprint
- rviz/g1_nav.rviz: update LiDAR PointCloud2 display settings

File: src/g1_description/g1_23dof.urdf (robot description, URDF)
Before this commit: robot g1_23dof, 33 links, 32 joints
Links:
- added link base_footprint
- added link lidar_link
- link head_link: geometry collision mesh filename=package://g1_description/meshes/head_link.STL; visual mesh filename=package://g1_description/meshes/head_link.STL
- link left_ankle_pitch_link: geometry collision mesh filename=package://g1_description/meshes/left_ankle_pitch_link.STL; visual mesh filename=package://g1_description/meshes/left_ankle_pitch_link.STL
- link left_ankle_roll_link: geometry collision sphere radius=0.005; collision sphere radius=0.005
- link left_elbow_link: geometry collision mesh filename=package://g1_description/meshes/left_elbow_link.STL; visual mesh filename=package://g1_description/meshes/left_elbow_link.STL
- link left_hip_pitch_link: geometry collision mesh filename=package://g1_description/meshes/left_hip_pitch_link.STL; visual mesh filename=package://g1_description/meshes/left_hip_pitch_link.STL
- link left_hip_roll_link: geometry collision mesh filename=package://g1_description/meshes/left_hip_roll_link.STL; visual mesh filename=package://g1_description/meshes/left_hip_roll_link.STL
- link left_hip_yaw_link: geometry collision mesh filename=package://g1_description/meshes/left_hip_yaw_link.STL; visual mesh filename=package://g1_description/meshes/left_hip_yaw_link.STL
- link left_knee_link: geometry collision mesh filename=package://g1_description/meshes/left_knee_link.STL; visual mesh filename=package://g1_description/meshes/left_knee_link.STL
- link left_shoulder_pitch_link: geometry collision cylinder length=0.05 radius=0.03; visual mesh filename=package://g1_description/meshes/left_shoulder_pitch_link.STL
- link left_shoulder_roll_link: geometry collision cylinder length=0.03 radius=0.03; visual mesh filename=package://g1_description/meshes/left_shoulder_roll_link.STL
- link left_shoulder_yaw_link: geometry collision mesh filename=package://g1_description/meshes/left_shoulder_yaw_link.STL; visual mesh filename=package://g1_description/meshes/left_shoulder_yaw_link.STL
- link left_wrist_roll_rubber_hand: geometry collision mesh filename=package://g1_description/meshes/left_wrist_roll_rubber_hand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; visual mesh filename=package://g1_description/meshes/left_wrist_roll_rubber_hand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
- link logo_link: geometry collision mesh filename=package://g1_description/meshes/logo_link.STL; visual mesh filename=package://g1_description/meshes/logo_link.STL
- link pelvis: geometry visual mesh filename=package://g1_description/meshes/pelvis.STL
- link pelvis_contour_link: geometry collision mesh filename=package://g1_description/meshes/pelvis_contour_link.STL; visual mesh filename=package://g1_description/meshes/pelvis_contour_link.STL
- link right_ankle_pitch_link: geometry collision mesh filename=package://g1_description/meshes/right_ankle_pitch_link.STL; visual mesh filename=package://g1_description/meshes/right_ankle_pitch_link.STL
- link right_ankle_roll_link: geometry collision sphere radius=0.005; collision sphere radius=0.005
- link right_elbow_link: geometry collision mesh filename=package://g1_description/meshes/right_elbow_link.STL; visual mesh filename=package://g1_description/meshes/right_elbow_link.STL
- link right_hip_pitch_link: geometry collision mesh filename=package://g1_description/meshes/right_hip_pitch_link.STL; visual mesh filename=package://g1_description/meshes/right_hip_pitch_link.STL
- link right_hip_roll_link: geometry collision mesh filename=package://g1_description/meshes/right_hip_roll_link.STL; visual mesh filename=package://g1_description/meshes/right_hip_roll_link.STL
- link right_hip_yaw_link: geometry collision mesh filename=package://g1_description/meshes/right_hip_yaw_link.STL; visual mesh filename=package://g1_description/meshes/right_hip_yaw_link.STL
- link right_knee_link: geometry collision mesh filename=package://g1_description/meshes/right_knee_link.STL; visual mesh filename=package://g1_description/meshes/right_knee_link.STL
- link right_shoulder_pitch_link: geometry collision cylinder length=0.05 radius=0.03; visual mesh filename=package://g1_description/meshes/right_shoulder_pitch_link.S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
- link right_shoulder_roll_link: geometry collision cylinder length=0.03 radius=0.03; visual mesh filename=package://g1_description/meshes/right_shoulder_roll_link.STL
- link right_shoulder_yaw_link: geometry collision mesh filename=package://g1_description/meshes/right_shoulder_yaw_link.STL; visual mesh filename=package://g1_description/meshes/right_shoulder_yaw_link.STL
- link right_wrist_roll_rubber_hand: geometry collision mesh filename=package://g1_description/meshes/right_wrist_roll_rubber_han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; visual mesh filename=package://g1_description/meshes/right_wrist_roll_rubber_han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
- link torso_link: geometry collision mesh filename=package://g1_description/meshes/torso_link.STL; visual mesh filename=package://g1_description/meshes/torso_link.STL
- link waist_support_link: geometry collision mesh filename=package://g1_description/meshes/waist_support_link.STL; visual mesh filename=package://g1_description/meshes/waist_support_link.STL
- link waist_yaw_fixed_link: geometry visual mesh filename=package://g1_description/meshes/waist_yaw_link.STL
Joints:
- added joint base_footprint_joint: type fixed, parent base_footprint, child pelvis, origin xyz=0 0 0.76 rpy=0 0 0
- added joint lidar_joint: type fixed, parent pelvis, child lidar_link, origin xyz=0 0 0.3 rpy=0 0 0
